File: Kicad/Main_board/Main_board.kicad_pcb (KiCad board)
At the start: 2 copper layers, 100 x 100 mm, 28 parts, among them J1 LIPO 2S, J10 DIST_FRONT, J11 SENSORES_LINEA, J12 DIST_DCHA, J2 MOT_IZQ, J3 TB6612FNG_A, J4 TB6612FNG_B, J5 DC-DC_5V, J6 HC-05, J7 MOT_DER, J8 DIST_IZQ, J9 CAMARA, SW1 SW_DPDT, SW2 SW_Push, SW3 SW_Push, U1 PCF8574

Commit message: Resistors modified
Parts:
- R1, R2: value 1k -> 220
Changed lines of the file:
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@@
     (links 90)
     (no_connects 0)
-    (area 99.899999 44.8 200.100001 150.100001)
+    (area 99.924999 49.924999 200.075001 150.075001)
     (thickness 1.6)
     (drawings 120)
@@
       (effects (font (size 1 1) (thickness 0.15)))
     )
-    (fp_text value 1k (at 5.08 2.31) (layer F.Fab)
+    (fp_text value 220 (at 5.08 2.31) (layer F.Fab)
       (effects (font (size 1 1) (thickness 0.15)))
     )
@@
       (effects (font (size 1 1) (thickness 0.15)))
     )
-    (fp_text value 1k (at 5.08 2.31 180) (layer F.Fab)
-      (effects (font (size 1 1) (thickness 0.15)))
-    )
+    (fp_text value 220 (at 5.08 2.31 180) (layer F.Fab)
+      (effects (font (size 1 1) (thickness 0.15)))
+    )

Commit message: DC-DC enable modified
Connections:
- J5 pad 1: +5V -> Net-(J5-Pad1)
Routing:
- net +5V: track 271.2 -> 269.3 mm
Other:
- outline, holes or cut-outs redrawn
Changed lines of the file:
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@@
 (kicad_pcb (version 4) (host pcbnew 4.0.6)
   (general
-    (links 90)
+    (links 89)
     (no_connects 0)
     (area 99.924999 49.924999 200.075001 150.075001)
     (thickness 1.6)
-    (drawings 120)
-    (tracks 423)
+    (drawings 124)
+    (tracks 421)
     (zones 0)
     (modules 28)
-    (nets 53)
+    (nets 54)
   )
   (page A4)
@@
   (net 51 ENC_DER_A)
   (net 52 ENC_DER_B)
+  (net 53 "Net-(J5-Pad1)")
   (net_class Default "Esta es la clase de red por defecto."
     (clearance 0.2)
@@
     (add_net ENC_IZQ_A)
     (add_net ENC_IZQ_B)
+    (add_net "Net-(J5-Pad1)")
   )
   (net_class "Bat supply" ""
@@
     )
     (pad 1 thru_hole rect (at 0 0 180) (size 1.7 1.7) (drill 1) (layers *.Cu *.Mask)
-      (net 18 +5V))
+      (net 53 "Net-(J5-Pad1)"))
     (pad 2 thru_hole oval (at 0 2.54 180) (size 1.7 1.7) (drill 1) (layers *.Cu *.Mask)
       (net 41 VDD))
@@
     )
   )
+  (gr_line (start 161 50) (end 163 50) (layer Edge.Cuts) (width 0.15))
+  (gr_line (start 137 50) (end 139 50) (layer Edge.Cuts) (width 0.15))
+  (gr_line (start 159 52) (end 161 50) (layer Edge.Cuts) (width 0.15))
+  (gr_line (start 141 52) (end 159 52) (layer Edge.Cuts) (width 0.15))
+  (gr_line (start 139 50) (end 141 52) (layer Edge.Cuts) (width 0.15))
   (gr_line (start 102.9 85.5) (end 118.5 60.4) (layer Dwgs.User) (width 0.15))
   (gr_line (start 102.9 85.5) (end 114.4 92.6) (layer Dwgs.User) (width 0.15))
@@
     (effects (font (size 3 3) (thickness 0.5)) (justify mirror))
   )
-  (gr_line (start 137 50) (end 163 50) (layer Edge.Cuts) (width 0.15))
   (gr_line (start 200 102.8) (end 168 55) (layer Edge.Cuts) (width 0.15))
   (gr_arc (start 163 55) (end 163 50) (angle 90) (layer Edge.Cuts) (width 0.15))
@@
   (via (at 116.6 110.2) (size 0.6) (drill 0.4) (layers F.Cu B.Cu) (net 18))
   (segment (start 116.6 110.2) (end 116.6 104.52) (width 0.5) (layer F.Cu) (net 18))
-  (segment (start 118.5 110.24) (end 116.64 110.24) (width 0.5) (layer F.Cu) (net 18))
-  (segment (start 116.64 110.24) (end 116.6 110.2) (width 0.5) (layer F.Cu) (net 18))
   (segment (start 116.6 104.52) (end 118.5 102.62) (width 0.5) (layer F.Cu) (net 18))
   (segment (start 164.6 74.046447) (end 164.6 74.4) (width 0.3048) (layer F.Cu) (net 19))
