File: hw/Kicad/Main_board_V2/Main_board.sch (KiCad schematic (older format))
At the start: 30 parts, among them J1 LIPO 2S, J10 DIST_FRONT, J11 SENSORES_LINEA, J12 DIST_DCHA, J2 MOT_IZQ, J3 TB6612FNG_A, J4 TB6612FNG_B, J5 DC-DC_5V, J6 HC-05, J7 MOT_DER, J8 DIST_IZQ, J9 CAMARA, SW1 SW_DPDT, SW2 SW_Push, SW3 SW_Push, U1 PCF8574

Commit message: Cambiado valor del diodo D4
Parts:
- D4: value 1N4001 -> 1N4148
Changed lines of the file:
@@
 LIBS:contrib
 LIBS:valves
-LIBS:switches
-LIBS:modules
 LIBS:switches2
 LIBS:Main_board-cache
@@
 Sheet 1 1
 Title "Main Board robot de carreras educativo"
-Date "2018-01-20"
+Date "2018-01-30"
 Rev "V2"
 Comp "Liga Nacional de Robótica de Competición"
@@
 P 4550 4800
 F 0 "D4" H 4550 4700 50  0000 C CNN
-F 1 "1N4001" H 4550 4600 50  0000 C CNN
+F 1 "1N4148" H 4550 4600 50  0000 C CNN
 F 2 "Diodes_THT:D_A-405_P10.16mm_Horizontal" H 4550 4800 50  0001 C CNN
 F 3 "" H 4550 4800 50  0001 C CNN

Commit message: PCBs adapted with Kicad libraries models
Parts:
- removed SW1: SW_DPDT, Main_board:switch_DPDT, symbol SW_DPDT
- added SW1: SW_DPDT, Main_board:SW_CuK_JS202011CQN_DPDT_Straight, symbol SW_DPDT_x2
- A1: footprint Modules:Arduino_Nano -> Main_board:Arduino_Nano
- D1, D2: footprint LEDs:LED_D3.0mm -> Main_board:LED_D3.0mm
- D3, D4: footprint Diodes_THT:D_A-405_P10.16mm_Horizontal -> Main_board:D_A-405_P10.16mm_Horizontal
- J1: footprint Connectors_JST:JST_XH_B03B-XH-A_03x2.50mm_Straight -> Main_board:JST_XH_B03B-XH-A_1x03_P2.50mm_Vertical
- J10, J12, J8: footprint Socket_Strips:Socket_Strip_Straight_1x03_Pitch2.00mm -> Main_board:PinHeader_1x03_P2.00mm_Vertical
- J11: footprint Socket_Strips:Socket_Strip_Angled_1x07_Pitch2.54mm -> Main_board:PinSocket_1x07_P2.54mm_Horizontal
- J2, J7: footprint Socket_Strips:Socket_Strip_Straight_1x06_Pitch2.00mm -> Main_board:PinHeader_1x06_P2.00mm_Vertical
- J3, J4: footprint Socket_Strips:Socket_Strip_Straight_1x08_Pitch2.54mm -> Main_board:PinSocket_1x08_P2.54mm_Vertical
- J5: footprint Socket_Strips:Socket_Strip_Angled_1x04_Pitch2.54mm -> Main_board:PinSocket_1x04_P2.54mm_Horizontal
- J6: footprint Socket_Strips:Socket_Strip_Straight_1x06_Pitch2.54mm -> Main_board:PinSocket_1x06_P2.54mm_Vertical
- J9: footprint Socket_Strips:Socket_Strip_Straight_1x05_Pitch2.54mm -> Main_board:PinHeader_1x05_P2.54mm_Vertical
- JP1: footprint Connectors:GS2 -> Main_board:SolderJumper-2_P1.3mm_Open_Pad1.0x1.5mm
- R1, R2, R3, R4, R5, R6, R7, R8: footprint Resistors_THT:R_Axial_DIN0207_L6.3mm_D2.5mm_P10.16mm_Horizontal -> Main_board:R_Axial_DIN0207_L6.3mm_D2.5mm_P10.16mm_Horizontal
- SW2, SW3: footprint Buttons_Switches_THT:SW_PUSH_6mm -> Main_board:SW_PUSH_6mm
- U1: footprint Housings_DIP:DIP-16_W7.62mm_LongPads -> Main_board:DIP-16_W7.62mm_Socket_LongPads
Connections:
- net +5V: now also SW1.5 (B)
- net +BATT: now also SW1.2 (B)
- net STBY_MOT: now also SW1.4 (A)
- net VDD: now also SW1.1 (A)
