File: hw/Kicad/Sensors_board_V2/Sensors_board.kicad_pcb (KiCad board)
At the start: 2 copper layers, 89.3 x 38.6 mm, 22 parts, among them J1 SENSORES_LINEA, U1 CNY70, U2 CNY70, U3 CNY70, U4 CNY70, U5 CNY70, U6 CNY70, U7 CNY70, U8 CNY70, U9 4052

Commit message: Included CD4052 socket
Parts:
- U9: footprint Package_DIP:DIP-16_W7.62mm_LongPads -> Package_DIP:DIP-16_W7.62mm_Socket_LongPads
Changed lines of the file:
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@@
     (add_net "Net-(R7-Pad2)")
-  )
-  (module Package_DIP:DIP-16_W7.62mm_LongPads (layer F.Cu)
-    (at 140.36 60.3 270)
-    (descr "16-lead though-hole mounted DIP package, row spacing 7.62 mm (300 mils), LongPads")
-    (tags "THT DIP DIL PDIP 2.54mm 7.62mm 300mil LongPads")
-    (fp_text reference U9 (at 3.81 -2.33 270) (layer F.SilkS)
-      (effects (font (size 1 1) (thickness 0.15)))
-    )
-    (fp_text value 4052 (at 3.81 20.11 270) (layer F.Fab)
-      (effects (font (size 1 1) (thickness 0.15)))
-    )
-    (fp_arc (start 3.81 -1.33) (end 2.81 -1.33) (angle -180) (layer F.SilkS) (width 0.12))
-    (fp_line (start 1.635 -1.27) (end 6.985 -1.27) (layer F.Fab) (width 0.1))
-    (fp_line (start 6.985 -1.27) (end 6.985 19.05) (layer F.Fab) (width 0.1))
-    (fp_line (start 6.985 19.05) (end 0.635 19.05) (layer F.Fab) (width 0.1))
-    (fp_line (start 0.635 19.05) (end 0.635 -0.27) (layer F.Fab) (width 0.1))
-    (fp_line (start 0.635 -0.27) (end 1.635 -1.27) (layer F.Fab) (width 0.1))
-    (fp_line (start 2.81 -1.33) (end 1.56 -1.33) (layer F.SilkS) (width 0.12))
-    (fp_line (start 1.56 -1.33) (end 1.56 19.11) (layer F.SilkS) (width 0.12))
-    (fp_line (start 1.56 19.11) (end 6.06 19.11) (layer F.SilkS) (width 0.12))
-    (fp_line (start 6.06 19.11) (end 6.06 -1.33) (layer F.SilkS) (width 0.12))
-    (fp_line (start 6.06 -1.33) (end 4.81 -1.33) (layer F.SilkS) (width 0.12))
-    (fp_line (start -1.45 -1.55) (end -1.45 19.3) (layer F.CrtYd) (width 0.05))
-    (fp_line (start -1.45 19.3) (end 9.1 19.3) (layer F.CrtYd) (width 0.05))
-    (fp_line (start 9.1 19.3) (end 9.1 -1.55) (layer F.CrtYd) (width 0.05))
-    (fp_line (start 9.1 -1.55) (end -1.45 -1.55) (layer F.CrtYd) (width 0.05))
-    (fp_text user %R (at 3.81 8.89 270) (layer F.Fab)
-      (effects (font (size 1 1) (thickness 0.15)))
-    )
-    (pad 1 thru_hole rect (at 0 0 270) (size 2.4 1.6) (drill 0.8) (layers *.Cu *.Mask)
-      (net 10 SENSOR_5))
-    (pad 9 thru_hole oval (at 7.62 17.78 270) (size 2.4 1.6) (drill 0.8) (layers *.Cu *.Mask)
-      (net 18 LINEA_SEL_2))
-    (pad 2 thru_hole oval (at 0 2.54 270) (size 2.4 1.6) (drill 0.8) (layers *.Cu *.Mask)
-      (net 21 SENSOR_7))
-    (pad 10 thru_hole oval (at 7.62 15.24 270) (size 2.4 1.6) (drill 0.8) (layers *.Cu *.Mask)
-      (net 5 LINEA_SEL_1))
-    (pad 3 thru_hole oval (at 0 5.08 270) (size 2.4 1.6) (drill 0.8) (layers *.Cu *.Mask)
-      (net 4 LINEA_2))
-    (pad 11 thru_hole oval (at 7.62 12.7 270) (size 2.4 1.6) (drill 0.8) (layers *.Cu *.Mask)
-      (net 9 SENSOR_4))
-    (pad 4 thru_hole oval (at 0 7.62 270) (size 2.4 1.6) (drill 0.8) (layers *.Cu *.Mask)
-      (net 22 SENSOR_8))
-    (pad 12 thru_hole oval (at 7.62 10.16 270) (size 2.4 1.6) (drill 0.8) (layers *.Cu *.Mask)
-      (net 6 SENSOR_1))
-    (pad 5 thru_hole oval (at 0 10.16 270) (size 2.4 1.6) (drill 0.8) (layers *.Cu *.Mask)
-      (net 11 SENSOR_6))
-    (pad 13 thru_hole oval (at 7.62 7.62 270) (size 2.4 1.6) (drill 0.8) (layers *.Cu *.Mask)
-      (net 3 LINEA_1))
-    (pad 6 thru_hole oval (at 0 12.7 270) (size 2.4 1.6) (drill 0.8) (layers *.Cu *.Mask)
-      (net 2 GND))
-    (pad 14 thru_hole oval (at 7.62 5.08 270) (size 2.4 1.6) (drill 0.8) (layers *.Cu *.Mask)
-      (net 7 SENSOR_2))
-    (pad 7 thru_hole oval (at 0 15.24 270) (size 2.4 1.6) (drill 0.8) (layers *.Cu *.Mask)
-      (net 2 GND))
-    (pad 15 thru_hole oval (at 7.62 2.54 270) (size 2.4 1.6) (drill 0.8) (layers *.Cu *.Mask)
-      (net 8 SENSOR_3))
-    (pad 8 thru_hole oval (at 0 17.78 270) (size 2.4 1.6) (drill 0.8) (layers *.Cu *.Mask)
-      (net 2 GND))
-    (pad 16 thru_hole oval (at 7.62 0 270) (size 2.4 1.6) (drill 0.8) (layers *.Cu *.Mask)
-      (net 1 +5V))
-    (model ${KISYS3DMOD}/Package_DIP.3dshapes/DIP-16_W7.62mm.wrl
-      (at (xyz 0 0 0))
-      (scale (xyz 1 1 1))
-      (rotate (xyz 0 0 0))
-    )
   )
   (module Sensors_board:PinHeader_1x07_P2.54mm_Horizontal (layer F.Cu)
@@
       (at (xyz 0 0 0))
       (scale (xyz 1 1 1))
+      (rotate (xyz 0 0 0))
+    )
+  )
+  (module Package_DIP:DIP-16_W7.62mm_Socket_LongPads (layer F.Cu)
+    (at 140.36 60.3 270)
+    (descr "16-lead though-hole mounted DIP package, row spacing 7.62 mm (300 mils), Socket, LongPads")
+    (tags "THT DIP DIL PDIP 2.54mm 7.62mm 300mil Socket LongPads")
+    (fp_text reference U9 (at 3.81 -2.33 270) (layer F.SilkS)
+      (effects (font (size 1 1) (thickness 0.15)))
+    )
+    (fp_text value 4052 (at 3.81 20.11 270) (layer F.Fab)
+      (effects (font (size 1 1) (thickness 0.15)))
+    )
+    (fp_arc (start 3.81 -1.33) (end 2.81 -1.33) (angle -180) (layer F.SilkS) (width 0.12))
+    (fp_line (start 1.635 -1.27) (end 6.985 -1.27) (layer F.Fab) (width 0.1))
+    (fp_line (start 6.985 -1.27) (end 6.985 19.05) (layer F.Fab) (width 0.1))
+    (fp_line (start 6.985 19.05) (end 0.635 19.05) (layer F.Fab) (width 0.1))
+    (fp_line (start 0.635 19.05) (end 0.635 -0.27) (layer F.Fab) (width 0.1))
+    (fp_line (start 0.635 -0.27) (end 1.635 -1.27) (layer F.Fab) (width 0.1))
+    (fp_line (start -1.27 -1.33) (end -1.27 19.11) (layer F.Fab) (width 0.1))
+    (fp_line (start -1.27 19.11) (end 8.89 19.11) (layer F.Fab) (width 0.1))
+    (fp_line (start 8.89 19.11) (end 8.89 -1.33) (layer F.Fab) (width 0.1))
+    (fp_line (start 8.89 -1.33) (end -1.27 -1.33) (layer F.Fab) (width 0.1))
+    (fp_line (start 2.81 -1.33) (end 1.56 -1.33) (layer F.SilkS) (width 0.12))
+    (fp_line (start 1.56 -1.33) (end 1.56 19.11) (layer F.SilkS) (width 0.12))
+    (fp_line (start 1.56 19.11) (end 6.06 19.11) (layer F.SilkS) (width 0.12))
+    (fp_line (start 6.06 19.11) (end 6.06 -1.33) (layer F.SilkS) (width 0.12))
+    (fp_line (start 6.06 -1.33) (end 4.81 -1.33) (layer F.SilkS) (width 0.12))
+    (fp_line (start -1.44 -1.39) (end -1.44 19.17) (layer F.SilkS) (width 0.12))
+    (fp_line (start -1.44 19.17) (end 9.06 19.17) (layer F.SilkS) (width 0.12))
+    (fp_line (start 9.06 19.17) (end 9.06 -1.39) (layer F.SilkS) (width 0.12))
+    (fp_line (start 9.06 -1.39) (end -1.44 -1.39) (layer F.SilkS) (width 0.12))
+    (fp_line (start -1.55 -1.6) (end -1.55 19.4) (layer F.CrtYd) (width 0.05))
+    (fp_line (start -1.55 19.4) (end 9.15 19.4) (layer F.CrtYd) (width 0.05))
+    (fp_line (start 9.15 19.4) (end 9.15 -1.6) (layer F.CrtYd) (width 0.05))
+    (fp_line (start 9.15 -1.6) (end -1.55 -1.6) (layer F.CrtYd) (width 0.05))
+    (fp_text user %R (at 3.81 8.89 270) (layer F.Fab)
+      (effects (font (size 1 1) (thickness 0.15)))
+    )
+    (pad 1 thru_hole rect (at 0 0 270) (size 2.4 1.6) (drill 0.8) (layers *.Cu *.Mask)
+      (net 10 SENSOR_5))
+    (pad 9 thru_hole oval (at 7.62 17.78 270) (size 2.4 1.6) (drill 0.8) (layers *.Cu *.Mask)
+      (net 18 LINEA_SEL_2))
+    (pad 2 thru_hole oval (at 0 2.54 270) (size 2.4 1.6) (drill 0.8) (layers *.Cu *.Mask)
+      (net 21 SENSOR_7))
+    (pad 10 thru_hole oval (at 7.62 15.24 270) (size 2.4 1.6) (drill 0.8) (layers *.Cu *.Mask)
+      (net 5 LINEA_SEL_1))
+    (pad 3 thru_hole oval (at 0 5.08 270) (size 2.4 1.6) (drill 0.8) (layers *.Cu *.Mask)
+      (net 4 LINEA_2))
+    (pad 11 thru_hole oval (at 7.62 12.7 270) (size 2.4 1.6) (drill 0.8) (layers *.Cu *.Mask)
+      (net 9 SENSOR_4))
+    (pad 4 thru_hole oval (at 0 7.62 270) (size 2.4 1.6) (drill 0.8) (layers *.Cu *.Mask)
+      (net 22 SENSOR_8))
+    (pad 12 thru_hole oval (at 7.62 10.16 270) (size 2.4 1.6) (drill 0.8) (layers *.Cu *.Mask)
+      (net 6 SENSOR_1))
+    (pad 5 thru_hole oval (at 0 10.16 270) (size 2.4 1.6) (drill 0.8) (layers *.Cu *.Mask)
+      (net 11 SENSOR_6))
+    (pad 13 thru_hole oval (at 7.62 7.62 270) (size 2.4 1.6) (drill 0.8) (layers *.Cu *.Mask)
+      (net 3 LINEA_1))
+    (pad 6 thru_hole oval (at 0 12.7 270) (size 2.4 1.6) (drill 0.8) (layers *.Cu *.Mask)
+      (net 2 GND))
+    (pad 14 thru_hole oval (at 7.62 5.08 270) (size 2.4 1.6) (drill 0.8) (layers *.Cu *.Mask)
+      (net 7 SENSOR_2))
+    (pad 7 thru_hole oval (at 0 15.24 270) (size 2.4 1.6) (drill 0.8) (layers *.Cu *.Mask)
+      (net 2 GND))
+    (pad 15 thru_hole oval (at 7.62 2.54 270) (size 2.4 1.6) (drill 0.8) (layers *.Cu *.Mask)
+      (net 8 SENSOR_3))
+    (pad 8 thru_hole oval (at 0 17.78 270) (size 2.4 1.6) (drill 0.8) (layers *.Cu *.Mask)
+      (net 2 GND))
+    (pad 16 thru_hole oval (at 7.62 0 270) (size 2.4 1.6) (drill 0.8) (layers *.Cu *.Mask)
+      (net 1 +5V))
+    (model ${KISYS3DMOD}/Package_DIP.3dshapes/DIP-16_W7.62mm_Socket.wrl
+      (at (xyz 0 0 0))
+      (scale (xyz 1 1 1))
