File: hw/Kicad/Sensors_board_V2/Sensors_board.sch (KiCad schematic (older format))
At the start: 17 parts, among them J1 SENSORES_LINEA, U1 CNY70, U2 CNY70, U3 CNY70, U4 CNY70, U5 CNY70, U6 CNY70, U7 4053

Commit message: Sensors_board_V2 Schematic, pdf and bom added
Parts:
- removed U7: 4053, Sensors_board:DIP-16_W7.62mm_Socket_LongPads, symbol 4053
- added R10: 82, Sensors_board:R_Axial_DIN0207_L6.3mm_D2.5mm_P10.16mm_Horizontal, symbol R
- added R11, R12: 10k, Sensors_board:R_Axial_DIN0207_L6.3mm_D2.5mm_P10.16mm_Horizontal, symbol R
- added U7, U8: CNY70, Sensors_board:Vishay_CNY70, symbol CNY70
- added U9: 4052, Package_DIP:DIP-16_W7.62mm_LongPads, symbol 4052
Connections:
- net labels added: LINEA_SEL_2, SENSOR_7, SENSOR_8
- net labels removed: LINEA_3
- wire segments 77 -> 92

Commit message: Included CD4052 socket
Parts:
- U9: footprint Package_DIP:DIP-16_W7.62mm_LongPads -> Package_DIP:DIP-16_W7.62mm_Socket_LongPads
Changed lines of the file:
@@
 F 0 "U9" H 8250 5250 50  0000 C CNN
 F 1 "4052" H 8250 5050 50  0000 C CNN
-F 2 "Package_DIP:DIP-16_W7.62mm_LongPads" H 8150 5250 60  0001 C CNN
+F 2 "Package_DIP:DIP-16_W7.62mm_Socket_LongPads" H 8150 5250 60  0001 C CNN
 F 3 "" H 8150 5250 60  0001 C CNN
 	1    8150 5250
